Commit message: New URDF

File: spotmicro/util/pybullet_data/assets/urdf/spot.urdf (robot description, URDF)
Before this commit: robot spot, 24 links, 23 joints
Links:
- added link cfr_core, mass 0.1; collision box size=0.048 0.145 0.026; visual mesh filename=package://mini_ros/stl/OpenQuadruped/cfr_core.stl scale=1 1 1
- added link m5paper, mass 0.1; collision box size=0.048 0.145 0.026; visual mesh filename=package://mini_ros/stl/OpenQuadruped/m5paper.stl scale=1 1 1
- added link m5paper2, mass 0.1; collision box size=0.048 0.145 0.026; visual mesh filename=package://mini_ros/stl/OpenQuadruped/lidar.stl scale=1 1 1
- link back: geometry collision box size=0.114 0.075 0.085; visual mesh filename=package://mini_ros/stl/OpenQuadruped/m5fire_black.stl scale=1 1 1
Joints:
- added joint base_cfr_core: type fixed, parent base_link, child cfr_core, origin xyz=-0.01 0 -0.0225 rpy=0 0 0
- added joint base_m5paper: type fixed, parent base_link, child m5paper, origin xyz=-0.01 0 -0.0225 rpy=0 0 0
- added joint base_m5paper2: type fixed, parent base_link, child m5paper2, origin xyz=-0.01 0 -0.0225 rpy=0 0 0

Commit message: new STLs right side

File: spotmicro/util/pybullet_data/assets/urdf/spot.urdf (robot description, URDF)
Before this commit: robot spot, 27 links, 26 joints
Links:
- link back_left_lower_leg: geometry collision box size=0.035 0.035 0.10; visual mesh filename=package://mini_ros/stl/OpenQuadruped/LEFT_LOWER_LEG.stl scale=1 1 1
- link back_right_lower_leg: geometry collision box size=0.035 0.035 0.10; visual mesh filename=package://mini_ros/stl/OpenQuadruped/RIGHT_LOWER_LEG.stl scale=1 1 1
- link front_left_lower_leg: geometry collision box size=0.035 0.035 0.10; visual mesh filename=package://mini_ros/stl/OpenQuadruped/LEFT_LOWER_LEG.stl scale=1 1 1
- link front_right_lower_leg: geometry collision box size=0.035 0.035 0.10; visual mesh filename=package://mini_ros/stl/OpenQuadruped/RIGHT_LOWER_LEG.stl scale=1 1 1

Commit message: Add IMU

File: spotmicro/util/pybullet_data/assets/urdf/spot.urdf (robot description, URDF)
Before this commit: robot spot, 27 links, 26 joints
Links:
- added link back_right_foot_IMU, mass 0.005; collision mesh filename=package://mini_ros/stl/OpenQuadruped/RIGHT_FOOT_IMU.stl scale=1 1 1; visual mesh filename=package://mini_ros/stl/OpenQuadruped/RIGHT_FOOT_IMU.stl scale=1 1 1
Joints:
- added joint back_right_leg_foot_IMU: type fixed, parent back_right_lower_leg, child back_right_foot_IMU, origin xyz=0 0 -0.1265 rpy=0 0 0

Commit message: IMU

File: spotmicro/util/pybullet_data/assets/urdf/spot.urdf (robot description, URDF)
Before this commit: robot spot, 28 links, 27 joints
Links:
- added link front_right_foot_IMU, mass 0.005; collision mesh filename=package://mini_ros/stl/OpenQuadruped/RIGHT_FOOT_IMU.stl scale=1 1 1; visual mesh filename=package://mini_ros/stl/OpenQuadruped/RIGHT_FOOT_IMU.stl scale=1 1 1
Joints:
- added joint front_right_leg_foot_IMU: type fixed, parent front_right_lower_leg, child front_right_foot_IMU, origin xyz=0 0 -0.1265 rpy=0 0 0

Commit message: add servos

File: spotmicro/util/pybullet_data/assets/urdf/spot.urdf (robot description, URDF)
Before this commit: robot spot, 29 links, 28 joints
Links:
- added link back_right_foot_CFP, mass 0.005; visual mesh filename=package://mini_ros/stl/OpenQuadruped/RIGHT_FOOT_CFP.stl scale=1 1 1
- added link back_right_foot_servo, mass 0.005; visual mesh filename=package://mini_ros/stl/OpenQuadruped/RIGHT_LOWER_SERVO.stl scale=1 1 1
- added link front_right_foot_CFP, mass 0.005; visual mesh filename=package://mini_ros/stl/OpenQuadruped/RIGHT_FOOT_CFP.stl scale=1 1 1
- added link front_right_foot_servo, mass 0.005; visual mesh filename=package://mini_ros/stl/OpenQuadruped/RIGHT_LOWER_SERVO.stl scale=1 1 1
- added link front_right_upper_servo, mass 0.005; visual mesh filename=package://mini_ros/stl/OpenQuadruped/RIGHT_UPPER_SERVO.stl scale=1 1 1
- link back_right_foot_IMU: geometry visual mesh filename=package://mini_ros/stl/OpenQuadruped/RIGHT_FOOT_IMU.stl scale=1 1 1
- link front_right_foot_IMU: geometry visual mesh filename=package://mini_ros/stl/OpenQuadruped/RIGHT_FOOT_IMU.stl scale=1 1 1
Joints:
- added joint back_right_leg_foot_CFP: type fixed, parent back_right_lower_leg, child back_right_foot_CFP, origin xyz=0 0 -0.1265 rpy=0 0 0
- added joint back_right_leg_foot_servo: type fixed, parent back_right_lower_leg, child back_right_foot_servo, origin xyz=0 0 -0.1265 rpy=0 0 0
- added joint front_right_leg_foot_CFP: type fixed, parent front_right_lower_leg, child front_right_foot_CFP, origin xyz=0 0 -0.1265 rpy=0 0 0
- added joint front_right_leg_foot_servo: type fixed, parent front_right_lower_leg, child front_right_foot_servo, origin xyz=0 0 -0.1265 rpy=0 0 0
- added joint front_right_leg_upper_servo: type fixed, parent front_right_upper_leg, child front_right_upper_servo, origin xyz=-0.005 -0.01 -0.235 rpy=0 0 0

Commit message: add RPI5.stl and OAKD_LITE.stl

File: spotmicro/util/pybullet_data/assets/urdf/spot.urdf (robot description, URDF)
Before this commit: robot spot, 34 links, 33 joints
Links:
- removed link m5paper2
- added link oak_d_lite, mass 0.1; collision box size=0.048 0.145 0.026; visual mesh filename=package://mini_ros/stl/OpenQuadruped/OAKD_LITE.stl scale=1 1 1
- added link rpi_5, mass 0.1; collision box size=0.048 0.145 0.026; visual mesh filename=package://mini_ros/stl/OpenQuadruped/RPI5.stl scale=1 1 1
- added link rpi_lidar, mass 0.1; collision box size=0.048 0.145 0.026; visual mesh filename=package://mini_ros/stl/OpenQuadruped/lidar.stl scale=1 1 1
Joints:
- removed joint base_m5paper2
- added joint base_oakd_lite: type fixed, parent base_link, child oak_d_lite, origin xyz=-0.01 0 -0.0225 rpy=0 0 0
- added joint base_rpi_5: type fixed, parent base_link, child rpi_5, origin xyz=-0.01 0 -0.0225 rpy=0 0 0
- added joint base_rpi_lidar: type fixed, parent base_link, child rpi_lidar, origin xyz=-0.01 0 -0.0225 rpy=0 0 0

Commit message: add insta360, r_upper_CFP

File: spotmicro/util/pybullet_data/assets/urdf/spot.urdf (robot description, URDF)
Before this commit: robot spot, 36 links, 35 joints
Links:
- added link front_right_upper_CFP, mass 0.005; visual mesh filename=package://mini_ros/stl/OpenQuadruped/RIGHT_UPPER_CFP.stl scale=1 1 1
- added link insta360, mass 0.1; collision box size=0.048 0.145 0.026; visual mesh filename=package://mini_ros/stl/OpenQuadruped/INSTA360.stl scale=1 1 1
Joints:
- added joint base_insta360: type fixed, parent base_link, child insta360, origin xyz=-0.01 0 -0.0225 rpy=0 0 0
- added joint front_right_upper_CFP: type fixed, parent front_right_upper_leg, child front_right_upper_CFP, origin xyz=-0.005 -0.01 -0.235 rpy=0 0 0
