Commit message: back_right leg

File: mini_ros/urdf/spot.urdf.xacro (robot description, xacro)
@@ -17,5 +17,5 @@
               width="0.2"
               height="0.1"
-              matname="orange"
+              matname="maroon"
               meshfile="package://mini_ros/stl/OpenQuadruped/MAINBODY.stl"
               meshscale="1 1 1" /> <!-- m to mm -->
@@ -32,28 +32,4 @@
               meshfile="package://mini_ros/stl/OpenQuadruped/Battery.stl"
               meshscale="1 1 1" /> <!-- m to mm -->
-  <!-- CHASSIS LEFT -->
-  <xacro:mesh_link name="chassis_left"
-              origin_rpy="0 ${pi/2} -${pi/2}" origin_xyz="0.016 0.003 0"
-              i_rpy="0 0 0" i_xyz="0 0 0"
-              mass="0.01"
-              c_xyz="0 0 0"
-              length="0.06"
-              width="0.15"
-              height="0.006"
-              matname="black"
-              meshfile="package://mini_ros/stl/OpenQuadruped/Chassis_Left_Side.stl"
-              meshscale="1 1 1" /> <!-- m to mm -->
-  <!-- CHASSIS Right -->
-  <xacro:mesh_link name="chassis_right"
-              origin_rpy="0 ${pi/2} ${pi/2}" origin_xyz="-0.016 -0.003 0"
-              i_rpy="0 0 0" i_xyz="0 0 0"
-              mass="0.01"
-              c_xyz="0 0 0"
-              length="0.06"
-              width="0.15"
-              height="0.006"
-              matname="black"
-              meshfile="package://mini_ros/stl/OpenQuadruped/Chassis_Right_Side.stl"
-              meshscale="1 1 1" /> <!-- m to mm -->
   <!-- FRONT -->
   <xacro:mesh_link name="front"
@@ -65,5 +41,5 @@
               width="0.045"
               height="0.085"
-              matname="orange"
+              matname="maroon"
               meshfile="package://mini_ros/stl/OpenQuadruped/Front.stl"
               meshscale="1 1 1" /> <!-- m to mm -->
@@ -77,6 +53,6 @@
               width="0.075"
               height="0.085"
-              matname="orange"
-              meshfile="package://mini_ros/stl/OpenQuadruped/Back.stl"
+              matname="black"
+              meshfile="package://mini_ros/stl/OpenQuadruped/m5fire_black.stl"
               meshscale="1 1 1" /> <!-- m to mm -->
   <!-- FRONT BRACKET -->
@@ -89,5 +65,5 @@
               width="0.075"
               height="0.085"
-              matname="black"
+              matname="maroon"
               meshfile="package://mini_ros/stl/OpenQuadruped/Front_Bracket.stl"
               meshscale="1 1 1" /> <!-- m to mm -->
@@ -101,5 +77,5 @@
               width="0.075"
               height="0.085"
-              matname="black"
+              matname="maroon"
               meshfile="package://mini_ros/stl/OpenQuadruped/Back_Bracket.stl"
               meshscale="1 1 1" /> <!-- m to mm -->
@@ -115,5 +91,5 @@
               width="0.065"
               height="0.065"
-              matname="black"
+              matname="white"
               meshfile="package://mini_ros/stl/OpenQuadruped/LEFT_HIP.stl"
               meshscale="1 1 1" /> <!-- m to mm -->
@@ -179,5 +155,5 @@
               height="0.065"
               radius="0.02"
-              matname="orange"
+              matname="maroon"
               meshfile="package://mini_ros/stl/OpenQuadruped/LEFT_FOOT.stl"
               meshscale="1 1 1" /> <!-- m to mm -->
@@ -195,5 +171,5 @@
               width="0.065"
               height="0.065"
-              matname="black"
+              matname="white"
               meshfile="package://mini_ros/stl/OpenQuadruped/LEFT_HIP.stl"
               meshscale="1 1 1" /> <!-- m to mm -->
@@ -259,5 +235,5 @@
               height="0.065"
               radius="0.02"
-              matname="orange"
+              matname="maroon"
               meshfile="package://mini_ros/stl/OpenQuadruped/LEFT_FOOT.stl"
               meshscale="1 1 1" /> <!-- m to mm -->
@@ -275,5 +251,5 @@
               width="0.065"
               height="0.065"
-              matname="black"
+              matname="white"
               meshfile="package://mini_ros/stl/OpenQuadruped/RIGHT_HIP.stl"
               meshscale="1 1 1" /> <!-- m to mm -->
@@ -339,5 +315,5 @@
               height="0.065"
               radius="0.02"
-              matname="orange"
+              matname="yellow"
               meshfile="package://mini_ros/stl/OpenQuadruped/RIGHT_FOOT.stl"
               meshscale="1 1 1" /> <!-- m to mm -->
@@ -348,17 +324,17 @@
   <!-- HIP -->
   <xacro:mesh_link name="back_right_hip"
-              origin_rpy="0 0 ${pi/2}" origin_xyz="-0.25 0.074 -0.067"
+              origin_rpy="0 0 ${pi/2}" origin_xyz="-0.258 0.074 -0.062"
               i_rpy="0 0 0" i_xyz="0 -0.075 0"
               mass="0.2"
-              c_xyz="0.015 ${-0.01} -0.01"
-              length="0.05"
-              width="0.065"
-              height="0.065"
-              matname="black"
+              c_xyz="0.015 ${-0.005} -0.01"
+              length="0.05"
+              width="0.065"
+              height="0.065"
+              matname="white"
               meshfile="package://mini_ros/stl/OpenQuadruped/RIGHT_HIP.stl"
               meshscale="1 1 1" /> <!-- m to mm -->
   <xacro:rev_joint name="motor_back_right_hip" type="revolute"
                     axis_xyz="1 0 0"
-                    origin_rpy="0 0 0" origin_xyz="${-0.2515+0.115} ${-(0.0044+0.035)} ${0.067-0.045}"
+                    origin_rpy="0 0 0" origin_xyz="${-0.1075} ${-(0.0044+0.035)} ${0.067-0.050}"
                     parent="back_bracket" child="back_right_hip"
                     effort="4.0" velocity="4.0"
@@ -369,17 +345,17 @@
   <!-- UPPER LEG -->
   <xacro:mesh_link name="back_right_upper_leg"
-              origin_rpy="0 0 ${pi/2}" origin_xyz="${-0.252} ${0.12} ${-0.055}"
-              i_rpy="0 0 0" i_xyz="-0.005 -0.0175 -0.055"
+              origin_rpy="0 0 ${pi/2}" origin_xyz="${-0.252} ${0.13} ${-0.053}"
+              i_rpy="0 0 0" i_xyz="-0.005 -0.017 -0.053"
               mass="0.13"
-              c_xyz="0 ${-0.02} -0.05"
-              length="0.035"
+              c_xyz="0 -0.01 -0.038"
+              length="0.045"
               width="0.035"
               height="0.11"
-              matname="black"
+              matname="maroon"
               meshfile="package://mini_ros/stl/OpenQuadruped/RIGHT_UPPER_LEG.stl"
               meshscale="1 1 1" /> <!-- m to mm -->
   <xacro:rev_joint name="motor_back_right_upper_leg" type="revolute"
                     axis_xyz="0 1 0"
-                    origin_rpy="0 0 0" origin_xyz="0.0015 -0.045 -0.0087"
+                    origin_rpy="0 0 0" origin_xyz="0.0015 -0.045 -0.011"
                     parent="back_right_hip" child="back_right_upper_leg"
                     effort="4.0" velocity="4.0"
@@ -388,4 +364,34 @@
                     lower="${-pi/2}"
                     upper="2.59"/>
+  <!-- UPPER SERVO -->
+  <xacro:c_less_mesh_link name="back_right_upper_servo"
+              origin_rpy="0 0 ${pi/2}" origin_xyz="${-0.252} ${0.13} ${-0.053}"
+              i_rpy="0 0 0" i_xyz="-0.005 -0.0175 -0.053"
+              mass="0.005"
+              c_xyz="0 ${-0.02} -0.05"
+              length="0.05"
+              width="0.065"
+              height="0.065"
+              matname="black"
+              meshfile="package://mini_ros/stl/OpenQuadruped/RIGHT_UPPER_SERVO.stl"
+              meshscale="1 1 1" /> <!-- m to mm -->
+  <xacro:frame_joint name="back_right_leg_upper_servo" type="fixed"
+                  origin_rpy="0 0 0" origin_xyz="0 0 0"
+                  parent="back_right_upper_leg" child="back_right_upper_servo"/>
+  <!-- UPPER CFP -->
+  <xacro:c_less_mesh_link name="back_right_upper_CFP"
+              origin_rpy="0 0 ${pi/2}" origin_xyz="${-0.252} ${0.13} ${-0.053}"
+              i_rpy="0 0 0" i_xyz="-0.005 -0.0175 -0.053"
+              mass="0.005"
+              c_xyz="0 ${-0.02} -0.05"
+              length="0.05"
+              width="0.065"
+              height="0.065"
+              matname="black"
+              meshfile="package://mini_ros/stl/OpenQuadruped/RIGHT_UPPER_CFP.stl"
+              meshscale="1 1 1" /> <!-- m to mm -->
+  <xacro:frame_joint name="back_right_leg_upper_CFP" type="fixed"
+                  origin_rpy="0 0 0" origin_xyz="0 0 0"
+                  parent="back_right_upper_leg" child="back_right_upper_CFP"/>
   <!-- LOWER LEG -->
   <xacro:mesh_link name="back_right_lower_leg"
@@ -393,14 +399,14 @@
               i_rpy="0 0 0" i_xyz="-0.01 0 -0.06"
               mass="0.05"
-              c_xyz="0 0 -0.06"
-              length="0.035"
-              width="0.035"
-              height="0.12"
-              matname="black"
+              c_xyz="0 -0.01 -0.04"
+              length="0.035"
+              width="0.035"
+              height="0.11"
+              matname="yellow"
               meshfile="package://mini_ros/stl/OpenQuadruped/RIGHT_LOWER_LEG.stl"
               meshscale="1 1 1" /> <!-- m to mm -->
   <xacro:rev_joint name="motor_back_right_lower_leg" type="revolute"
                     axis_xyz="0 1 0"
-                    origin_rpy="0 0 0" origin_xyz="-0.005 -0.018 -0.109"
+                    origin_rpy="0 0 0" origin_xyz="-0.005 -0.002 -0.1068"
                     parent="back_right_upper_leg" child="back_right_lower_leg"
                     effort="4.0" velocity="4.0"
@@ -409,10 +415,55 @@
                     lower="-2.9"
                     upper="${pi/2}"/>
+  <!-- LOWER SERVO -->
+  <xacro:c_less_mesh_link name="back_right_lower_servo"
+              origin_rpy="0 0 ${pi/2}" origin_xyz="${-0.247} ${0.1375} ${0.18}"
+              i_rpy="0 0 0" i_xyz="0 0 0"
+              mass="0.005"
+              c_xyz="${-0.247} ${0.138} ${0.18}"
+              length="0.05"
+              width="0.065"
+              height="0.065"
+              matname="black"
+              meshfile="package://mini_ros/stl/OpenQuadruped/RIGHT_LOWER_SERVO.stl"
+              meshscale="1 1 1" /> <!-- m to mm -->
+  <xacro:frame_joint name="back_right_leg_lower_servo" type="fixed"
+                  origin_rpy="0 0 0" origin_xyz="0 0 -0.1265"
+                  parent="back_right_lower_leg" child="back_right_lower_servo"/>
+  <!-- LOWER CFP -->
+  <xacro:c_less_mesh_link name="back_right_lower_CFP"
+              origin_rpy="0 0 ${pi/2}" origin_xyz="${-0.247} ${0.138} ${0.18}"
+              i_rpy="0 0 0" i_xyz="0 0 0"
+              mass="0.005"
+              c_xyz="${-0.247} ${0.138} ${0.18}"
+              length="0.05"
+              width="0.065"
+              height="0.065"
+              matname="black"
+              meshfile="package://mini_ros/stl/OpenQuadruped/RIGHT_LOWER_CFP.stl"
+              meshscale="1 1 1" /> <!-- m to mm -->
+  <xacro:frame_joint name="back_right_leg_lower_CFP" type="fixed"
+                  origin_rpy="0 0 0" origin_xyz="0 0 -0.1265"
+                  parent="back_right_lower_leg" child="back_right_lower_CFP"/>
+  <!-- IMU -->
+  <xacro:c_less_mesh_link name="back_right_lower_IMU"
+              origin_rpy="0 0 ${pi/2}" origin_xyz="${-0.247} ${0.138} ${0.18}"
+              i_rpy="0 0 0" i_xyz="0 0 0"
+              mass="0.005"
+              c_xyz="${-0.247} ${0.138} ${0.18}"
+              length="0.05"
+              width="0.065"
+              height="0.065"
+              matname="blue"
+              meshfile="package://mini_ros/stl/OpenQuadruped/RIGHT_FOOT_IMU.stl"
+              meshscale="1 1 1" /> <!-- m to mm -->
+  <xacro:frame_joint name="back_right_leg_lower_IMU" type="fixed"
+                  origin_rpy="0 0 0" origin_xyz="0 0 -0.1265"
+                  parent="back_right_lower_leg" child="back_right_lower_IMU"/>
   <!-- FOOT -->
   <xacro:mesh_link_sphere name="back_right_foot"
-              origin_rpy="0 0 ${pi/2}" origin_xyz="${-0.247} ${0.138} ${0.18}"
-              i_rpy="0 0 0" i_xyz="0 0 0"
-              mass="0.005"
-              c_xyz="${-0.247} ${0.138} ${0.18}"
+              origin_rpy="0 0 ${pi/2}" origin_xyz="${-0.247} ${0.138} ${0.1535}"
+              i_rpy="0 0 0" i_xyz="0 0 0"
+              mass="0.005"
+              c_xyz="${-0.247} ${0.138} ${0.1535}"
               length="0.05"
               width="0.065"
@@ -423,5 +474,5 @@
               meshscale="1 1 1" /> <!-- m to mm -->
   <xacro:frame_joint name="back_right_leg_foot" type="fixed"
-                  origin_rpy="0 0 0" origin_xyz="0 0 -0.1265"
+                  origin_rpy="0 0 0" origin_xyz="0 0 -0.1"
                   parent="back_right_lower_leg" child="back_right_foot"/>
 <!-- STATIC Joints -->
@@ -434,12 +485,4 @@
                   origin_rpy="0 0 0" origin_xyz="-0.01 0 -0.0225"
                   parent="base_link" child="battery"/>
-<!-- MAIN BODY TO CHASSIS LEFT -->
-<xacro:frame_joint name="base_left" type="fixed"
-                  origin_rpy="0 0 0" origin_xyz="0.00 0.052 0"
-                  parent="base_link" child="chassis_left"/>
-<!-- MAIN BODY TO CHASSIS RIGHT -->
-<xacro:frame_joint name="base_right" type="fixed"
-                  origin_rpy="0 0 0" origin_xyz="0.00 -0.052 0"
-                  parent="base_link" child="chassis_right"/>
 <!-- MAIN BODY TO FRONT -->
 <xacro:frame_joint name="base_front" type="fixed"

File: mini_ros/urdf/spot_macro.xacro (robot description, xacro)
@@ -1,13 +1,34 @@
 <?xml version="1.0" ?>
 <robot xmlns:xacro="http://www.ros.org/wiki/xacro">
-  <material name="orange">
-    <color rgba="1.0 0.5 0.0 1"/>
-  </material>
-  <material name="black">
-    <color rgba="0.1 0.1 0.1 1"/>
-  </material>
-  <material name="grey">
-    <color rgba="0.6 0.6 0.6 1"/>
-  </material>
+<material name="maroon">
+  <color rgba="0.5 0.2 0.2 1"/>
+</material>
+<material name="lblue">
+  <color rgba="0.1 0.1 0.8 0.9"/>
+</material>
+<material name="orange">
+  <color rgba="1.0 0.5 0.0 1"/>
+</material>
+<material name="black">
+  <color rgba="0.1 0.1 0.1 1"/>
+</material>
+<material name="grey">
+  <color rgba="0.6 0.6 0.6 1"/>
+</material>
+<material name="white">
+  <color rgba="1.0 1.0 1.0 1"/>
+</material>
+<material name="yellow">
+  <color rgba="1.0 1.0 0.0 1"/>
+</material>
+<material name="cgray">
+  <color rgba="0.6 0.6 0.6 0.5"/>
+</material>
+<material name="blue">
+  <color rgba="0.2 0.2 0.8 1"/>
+</material>
+<material name="green">
+  <color rgba="0.2 0.8 0.2 1"/>
+</material>
   <xacro:macro name="rev_joint" params="name type axis_xyz origin_rpy origin_xyz parent child effort velocity damping friction upper lower">
     <joint name="${name}" type="${type}">
@@ -53,5 +74,29 @@
         </xacro:if>
         <xacro:if value="${matname == 'orange'}">
-          <material>Gazebo/Orange</material>
+          <material>Gazebo/Red</material>
+        </xacro:if>
+    </gazebo>
+  </xacro:macro>
+  <xacro:macro name="c_less_mesh_link" params="name origin_xyz origin_rpy meshfile meshscale c_xyz matname mass i_xyz i_rpy length width height">
+    <link name="${name}">
+      <visual>
+        <origin rpy="${origin_rpy}" xyz="${origin_xyz}" />
+        <geometry>
+          <mesh filename="${meshfile}" scale="${meshscale}"/>
+        </geometry>
+        <material name="${matname}"/>
+      </visual>
+      <inertial>
+        <mass value="${mass}" />
+        <origin rpy="${i_rpy}" xyz="${i_xyz}" /> <!-- Inertial Axes -->
+        <inertia ixx="${mass * (width * width + height * height)/12.0}" ixy="${0}" ixz="${0}" iyx="${0}" iyy="${mass * (length * length + height * height)/12.0}" iyz="${0}" izx="${0}" izy="${0}" izz="${mass * (length * length + width * width)/12.0}" />
+      </inertial>
+    </link>
+    <gazebo reference="${name}">
+        <xacro:if value="${matname == 'black'}">
+          <material>Gazebo/Black</material>
+        </xacro:if>
+        <xacro:if value="${matname == 'orange'}">
+          <material>Gazebo/Red</material>
         </xacro:if>
     </gazebo>
@@ -86,5 +131,5 @@
       <maxVel>0.0</maxVel>
       <minDepth>0.001</minDepth>
-      <material>Gazebo/Orange</material>
+      <material>Gazebo/Red</material>
     </gazebo>
   </xacro:macro>
