Commit message: .xacro modifications

File: mini_ros/urdf/spot_macro.xacro (robot description, xacro)
@@ -5,5 +5,5 @@
 </material>
 <material name="lblue">
-  <color rgba="0.1 0.1 0.8 0.9"/>
+  <color rgba="0.01 0.01 0.08 0.7"/>
 </material>
 <material name="orange">
@@ -13,5 +13,5 @@
   <color rgba="0.1 0.1 0.1 1"/>
 </material>
-<material name="grey">
+<material name="gray">
   <color rgba="0.6 0.6 0.6 1"/>
 </material>
