Commit message: v10.5 PyBullet Working

File: mini_ros/urdf/spot.urdf (robot description, URDF)
Before this commit: robot spot, 25 links, 24 joints
Links:
- link front_right_lower_leg: geometry collision box size=0.035 0.035 0.11; visual mesh filename=package://mini_ros/stl/OpenQuadruped/RIGHT_LOWER_LEG.stl scale=1 1 1
Joints:
- joint motor_front_right_lower_leg: origin xyz=-0.005 -0.018 -0.109 rpy=0 0 0 -> xyz=-0.005 -0.002 -0.1068 rpy=0 0 0
- joint motor_front_right_upper_leg: origin xyz=0.0015 -0.045 -0.0087 rpy=0 0 0 -> xyz=0.0015 -0.045 -0.011 rpy=0 0 0
